Commit message: created the 5 dof, corrected flaws in the 3 dof

File: ros_ws/three_dof_robot_ws/src/welder_description/urdf/welder.xacro (robot description, xacro)
@@ -2,6 +2,14 @@
 <robot name="welder" xmlns:xacro="http://www.ros.org/wiki/xacro">
 <xacro:include filename="$(find welder_description)/urdf/materials.xacro" />
+<xacro:include filename="$(find welder_description)/urdf/ros2_control.xacro" />
 <xacro:include filename="$(find welder_description)/urdf/welder.trans" />
 <xacro:include filename="$(find welder_description)/urdf/welder.gazebo" />
+<link name="world">
+</link>
+<joint name="world" type="fixed">
+  <parent link="world"/>
+  <child link="base_link"/>
+  <origin xyz="0.0 0.0 0.0" rpy="0.0 0.0 0.0"/>
+</joint>
 <link name="base_link">
   <inertial>
@@ -84,64 +92,4 @@
   </collision>
 </link>
-<link name="link_4_1">
-  <inertial>
-    <origin xyz="0.0 -0.024901368509315194 0.031832335951871196" rpy="0 0 0"/>
-    <mass value="1.2085805984841382"/>
-    <inertia ixx="0.001374" iyy="0.001327" izz="0.000295" ixy="0.0" iyz="4e-06" ixz="0.0"/>
-  </inertial>
-  <visual>
-    <origin xyz="-0.0 0.075 -0.11" rpy="0 0 0"/>
-    <geometry>
-      <mesh filename="file://$(find welder_description)/meshes/link_4_1.stl" scale="0.001 0.001 0.001"/>
-    </geometry>
-    <material name="silver"/>
-  </visual>
-  <collision>
-    <origin xyz="-0.0 0.075 -0.11" rpy="0 0 0"/>
-    <geometry>
-      <mesh filename="file://$(find welder_description)/meshes/link_4_1.stl" scale="0.001 0.001 0.001"/>
-    </geometry>
-  </collision>
-</link>
-<link name="link_5_1">
-  <inertial>
-    <origin xyz="0.0 -4.404769588479962e-05 0.03489668781804081" rpy="0 0 0"/>
-    <mass value="0.7187100595069817"/>
-    <inertia ixx="0.000352" iyy="0.000343" izz="0.000159" ixy="-0.0" iyz="1e-06" ixz="0.0"/>
-  </inertial>
-  <visual>
-    <origin xyz="-0.0 0.1 -0.2" rpy="0 0 0"/>
-    <geometry>
-      <mesh filename="file://$(find welder_description)/meshes/link_5_1.stl" scale="0.001 0.001 0.001"/>
-    </geometry>
-    <material name="silver"/>
-  </visual>
-  <collision>
-    <origin xyz="-0.0 0.1 -0.2" rpy="0 0 0"/>
-    <geometry>
-      <mesh filename="file://$(find welder_description)/meshes/link_5_1.stl" scale="0.001 0.001 0.001"/>
-    </geometry>
-  </collision>
-</link>
-<link name="link_6_1">
-  <inertial>
-    <origin xyz="0.0 -0.01680268432280871 1.6653345369377348e-16" rpy="0 0 0"/>
-    <mass value="0.26501912859947435"/>
-    <inertia ixx="5.2e-05" iyy="3.9e-05" izz="5.2e-05" ixy="0.0" iyz="-0.0" ixz="-0.0"/>
-  </inertial>
-  <visual>
-    <origin xyz="-0.0 0.12 -0.25" rpy="0 0 0"/>
-    <geometry>
-      <mesh filename="file://$(find welder_description)/meshes/link_6_1.stl" scale="0.001 0.001 0.001"/>
-    </geometry>
-    <material name="silver"/>
-  </visual>
-  <collision>
-    <origin xyz="-0.0 0.12 -0.25" rpy="0 0 0"/>
-    <geometry>
-      <mesh filename="file://$(find welder_description)/meshes/link_6_1.stl" scale="0.001 0.001 0.001"/>
-    </geometry>
-  </collision>
-</link>
 <joint name="joint_1" type="continuous">
   <origin xyz="0.0 0.0 0.05" rpy="0 0 0"/>
@@ -162,21 +110,3 @@
   <axis xyz="0.0 0.0 -1.0"/>
 </joint>
-<joint name="joint_4" type="continuous">
-  <origin xyz="0.0 -0.025 -0.09" rpy="0 0 0"/>
-  <parent link="link_3_1"/>
-  <child link="link_4_1"/>
-  <axis xyz="0.0 1.0 0.0"/>
-</joint>
-<joint name="joint_5" type="continuous">
-  <origin xyz="0.0 -0.025 0.09" rpy="0 0 0"/>
-  <parent link="link_4_1"/>
-  <child link="link_5_1"/>
-  <axis xyz="0.0 0.0 1.0"/>
-</joint>
-<joint name="joint_6" type="continuous">
-  <origin xyz="0.0 -0.02 0.05" rpy="0 0 0"/>
-  <parent link="link_5_1"/>
-  <child link="link_6_1"/>
-  <axis xyz="0.0 -1.0 0.0"/>
-</joint>
 </robot>
