Commit message: update

File: Tests/gewnlimb_ws/src/gwenLimb_description/urdf/gwenLimb.xacro (robot description, xacro)
@@ -2,6 +2,16 @@
 <robot name="gwenLimb" xmlns:xacro="http://www.ros.org/wiki/xacro">
 <xacro:include filename="$(find gwenLimb_description)/urdf/materials.xacro" />
+<xacro:include filename="$(find gwenLimb_description)/urdf/ros2_control.xacro" />
 <xacro:include filename="$(find gwenLimb_description)/urdf/gwenLimb.trans" />
 <xacro:include filename="$(find gwenLimb_description)/urdf/gwenLimb.gazebo" />
+<link name="world">
+</link>
+<joint name="world_joint" type="fixed">
+  <origin xyz="0.0 0.0 0.0" rpy="0.0 0.0 0.0"/>
+  <parent link="world"/>
+  <child link="base_link"/>
+  <axis xyz="0.0 0.0 0.0"/>
+  <limit lower="0.0" upper="0.0" effort="0.0" velocity="0.0"/>
+</joint>
 <link name="base_link">
   <inertial>

File: Tests/gewnlimb_ws/src/gwenLimb_description/urdf/ros2_control.xacro (robot description, xacro)
@@ -2,6 +2,53 @@
 <robot name="gwenLimb" xmlns:xacro="http://www.ros.org/wiki/xacro" >
 <gazebo>
-  <plugin name="gazebo_ros2_control" filename="libgazebo_ros2_control.so"/>
+    <plugin name="gazebo_ros2_control" filename="libgazebo_ros2_control.so">
+        <robot_sim_type>gazebo_ros2_control/GazeboSystem</robot_sim_type>
+        <parameters>$(find gwenLimb_description)/config/robot_control.yaml</parameters>
+    </plugin>
 </gazebo>
-<ros2_control name = "Gwen Limb" type =
+<ros2_control name = "Gwen Limb" type = "system">
+    <hardware>
+        <plugin>gazebo_ros2_control/GazeboSystem</plugin>
+    </hardware>
+    <joint name="joint_1">
+        <command_interface name = "position">
+            <param name="min">-0.174533</param>
+            <param name="max">0.174533</param>
+        </command_interface>
+        <state_interface name = "position">
+            <param name = "initial_value">0.0</param>
+        </state_interface>
+        <state_interface name = "velocity"></state_interface>
+    </joint>
+    <joint name="joint_2">
+        <command_interface name = "position">
+            <param name="min">-1.047198</param>
+            <param name="max">1.047198</param>
+        </command_interface>
+        <state_interface name = "position">
+            <param name = "initial_value">0.0</param>
+        </state_interface>
+        <state_interface name = "velocity"></state_interface>
+    </joint>
+    <joint name="joint_3">
+        <command_interface name = "position">
+            <param name="min">-1.48353</param>
+            <param name="max">3.403392</param>
+        </command_interface>
+        <state_interface name = "position">
+            <param name = "initial_value">0.0</param>
+        </state_interface>
+        <state_interface name = "velocity"></state_interface>
+    </joint>
+    <joint name="joint_4">
+        <command_interface name = "position">
+            <param name="min">-3.14</param>
+            <param name="max">3.14</param>
+        </command_interface>
+        <state_interface name = "position">
+            <param name = "initial_value">0.0</param>
+        </state_interface>
+        <state_interface name = "velocity"></state_interface>
+    </joint>
+</ros2_control>
 </robot>
